Commit message: 나무없이

File: m0617_gripper/dsr_description2/urdf/m0617.urdf (robot description, URDF)
Before this commit: robot m0617, 8 links, 7 joints
Links:
- added link gripper_frame
Joints:
- added joint link_6-gripper_frame: type fixed, parent link_6, child gripper_frame, origin xyz=-0.018632895 -0.036789604 -0.118001442 rpy=-1.869670219 -0.156350649 -0.936767921
